File: src/IDC_50_PIN.sch (KiCad schematic (older format))
At the start: 28 parts, among them J1 EXPANSION, J10 Z1_Motor, J12 Z_STOP, J14 PANELDUE, J15 ESP_COMM, J17 Extruder_Heater, J18 LCD_CONN, J19 LCD_SD, J2 E1_STOP, J20 FAN2, J21 THERMISTOR2, J22 Z_PROBE, J23 FAN1, J24 THERMISTOR1, J25 FAN0, J26 ALWAYS_FAN1, J27 ALWAYS_FAN0, J28 THERMISTOR0, J3 E1_Motor, J4 E0_STOP, J5 E0_motor, J6 X_STOP, J7 X_motor, J8 Y_motor, J9 Y_STOP, M1 LOGO

Commit message: Test change
Parts:
- added M2, M3: FID, Fiducial:Fiducial_1mm_Mask3mm, symbol DuetWifi:FID
Changed lines of the file:
@@
 Wire Notes Line
 	2600 500  2600 10500
+$Comp
+L DuetWifi:FID M3
+U 1 1 6066E704
+P 1775 9400
+F 0 "M3" H 1853 9506 60  0000 L CNN
+F 1 "FID" H 1853 9400 60  0000 L CNN
+F 2 "Fiducial:Fiducial_1mm_Mask3mm" H 1853 9294 60  0000 L CNN
+F 3 "" H 1775 9400 60  0000 C CNN
+	1    1775 9400
+	1    0    0    -1
+$EndComp
+$Comp
+L DuetWifi:FID M2
+U 1 1 6066EC07
+P 1750 9775
+F 0 "M2" H 1828 9881 60  0000 L CNN
+F 1 "FID" H 1828 9775 60  0000 L CNN
+F 2 "Fiducial:Fiducial_1mm_Mask3mm" H 1828 9669 60  0000 L CNN
+F 3 "" H 1750 9775 60  0000 C CNN
+	1    1750 9775
+	1    0    0    -1
+$EndComp
 $EndSCHEMATC
