File: src/expansion.kicad_pcb (KiCad board)
At the start: 2 copper layers, 123.1 x 100.1 mm, 121 parts, among them J1 EXPANSION, J10 Z1_Motor, J12 Z_STOP, J14 PANELDUE, J15 ESP_COMM, J16 PANEL_DUE_OUT, J17 Extruder_Heater, J18 LCD_CONN, J19 LCD_SD, J2 E1_STOP, J20 FAN2, J21 THERMISTOR2, J22 Z_PROBE, J23 FAN1, J24 THERMISTOR1, J25 FAN0, J26 ALWAYS_FAN1, J27 ALWAYS_FAN0, J28 THERMISTOR0, J29 Conn_01x02, J3 E1_Motor, J30 Conn_01x02, J31 Conn_01x02, J32 Conn_01x02, J33 Conn_01x02, J34 Conn_01x02, J36 Z1, J37 Z1, J39 X, J4 E0_STOP, J40 Y2, J41 Y1, J42 Conn_02x20_Odd_Even, J43 Bed_Connections, J5 E0_motor, J6 X_STOP, J7 X_motor, J8 Y_motor, J9 Y_STOP, M1 LOGO, M3 FID, M4 MOUNTING, M5 MOUNTING, M6 MOUNTING, M7 MOUNTING, Q1 DMG2305UX-13, Q2 2N7002-7-F, Q3 DMG2305UX-13, Q4 2N7002-7-F, Q5 DMG2305UX-13, Q6 2N7002-7-F, U1 SN74HCT04PWR, U2 SN74HCT04PWR, U3 SN74HCT04PWR, U4 MC74VHCT50ADTR2G, U5 74HC14

Commit message: Test change
Parts:
- added M2: FID, Fiducial:Fiducial_1mm_Mask3mm, B.Cu at (137.4, 124.3)
- added M3: FID, Fiducial:Fiducial_1mm_Mask3mm, B.Cu at (150.0, 37.2)
Routing:
- net GND: vias 256 -> 273
Other:
- board text added: "Pantheon_10x_Shield_Rev2.7"
- board text removed: "Pantheon_10x_Shield_Rev2.6"

Commit message: Moved board
Parts:
- moved F6 19.0 mm to (143.8, 55.4)
- moved J14 19.0 mm to (143.0, 124.4)
- moved J3 19.0 mm to (128.0, 30.6)
- moved TP6 19.0 mm to (137.8, 75.5)
- moved TP7 19.0 mm to (133.3, 75.4)
- moved F2 19.0 mm to (70.9, 55.5)
- moved J26 19.0 mm to (73.9, 76.2)
- moved J30 19.0 mm to (74.9, 48.5)
- moved R27 19.0 mm to (79.2, 37.8)
- moved J28 19.0 mm to (50.5, 116.2)
- moved M3 19.0 mm to (49.7, 37.4)
- moved TP4 19.0 mm to (49.2, 111.0)
- moved C1 19.0 mm to (104.9, 76.2)
- moved C2 19.0 mm to (105.0, 73.7)
- moved C3 19.0 mm to (161.6, 55.0)
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
Commit message: Moved board again
Parts:
- moved F4 38.0 mm to (144.8, 56.0)
- moved J42 38.0 mm to (141.3, 89.8)
- moved J5 38.0 mm to (149.1, 31.2)
- moved M1 38.0 mm to (160.3, 106.0)
- moved Q2 38.0 mm to (136.3, 81.0)
- moved Q4 38.0 mm to (145.0, 80.2)
- moved Q6 38.0 mm to (156.0, 74.0)
- moved R26 38.0 mm to (135.3, 41.5)
- moved R32 38.0 mm to (163.6, 75.2)
- moved R8 38.0 mm to (154.1, 35.5)
- moved HS1 38.0 mm to (95.4, 123.8)
- moved C1 38.0 mm to (142.9, 76.8)
- moved C2 38.0 mm to (143.0, 74.2)
- moved C3 38.0 mm to (199.6, 55.5)
- moved C4 38.0 mm to (107.8, 105.2)
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
Commit message: Moved board last time
Parts:
- moved C1 11.8 mm to (154.7, 76.8)
- moved C2 11.8 mm to (154.7, 74.2)
- moved C3 11.8 mm to (211.3, 55.5)
- moved C4 11.8 mm to (119.6, 105.2)
- moved C5 11.8 mm to (112.5, 104.2)
- moved C6 11.8 mm to (140.1, 107.2)
- moved C7 11.8 mm to (131.0, 106.8)
- moved C8 11.8 mm to (167.2, 77.3)
- moved C9 11.8 mm to (164.9, 79.0)
- moved D1 11.8 mm to (200.1, 115.0)
- moved D2 11.8 mm to (200.0, 120.0)
- moved D4 11.8 mm to (151.4, 73.3)
- moved D5 11.8 mm to (106.8, 55.1)
- moved D6 11.8 mm to (203.2, 73.7)
- moved D7 11.8 mm to (210.9, 73.8)
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
Commit message: trace change
Routing:
- net E0-: track 279.4 -> 279.9 mm
Changed lines of the file:
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@@
   (segment (start 210.864982 30.724992) (end 210.880735 30.709239) (width 0.75) (layer F.Cu) (net 6))
   (segment (start 210.880735 30.709239) (end 210.880735 30.706482) (width 0.75) (layer F.Cu) (net 6))
-  (segment (start 210.287252 30.112999) (end 210.880735 30.706482) (width 0.75) (layer F.Cu) (net 6))
-  (segment (start 193.6 31.45) (end 194.937001 30.112999) (width 0.75) (layer F.Cu) (net 6) (status 10))
-  (segment (start 194.937001 30.112999) (end 210.287252 30.112999) (width 0.75) (layer F.Cu) (net 6))
   (segment (start 157.25 88.55) (end 166.124979 79.675021) (width 0.75) (layer F.Cu) (net 6))
   (segment (start 151.75 88.55) (end 157.25 88.55) (width 0.75) (layer F.Cu) (net 6))
@@
   (segment (start 166.700011 80.599989) (end 196.955908 80.599989) (width 0.75) (layer F.Cu) (net 6))
   (via (at 199.115054 82.759135) (size 0.8) (drill 0.4) (layers F.Cu B.Cu) (net 6))
-  (via (at 210.880735 30.706482) (size 0.8) (drill 0.4) (layers F.Cu B.Cu) (net 6) (status 1000000))
+  (via (at 210.880735 30.706482) (size 0.8) (drill 0.4) (layers F.Cu B.Cu) (net 6))
+  (segment (start 209.674253 29.5) (end 210.880735 30.706482) (width 0.75) (layer F.Cu) (net 6))
+  (segment (start 193.6 31.45) (end 195.55 29.5) (width 0.75) (layer F.Cu) (net 6))
+  (segment (start 195.55 29.5) (end 209.674253 29.5) (width 0.75) (layer F.Cu) (net 6))
   (segment (start 161.214998 66.498987) (end 161.214998 70.802498) (width 0.25) (layer B.Cu) (net 8))
   (segment (start 177.552989 66.099989) (end 161.613996 66.099989) (width 0.25) (layer B.Cu) (net 8))
